File: pcb.kicad_pcb (KiCad board)
At the start: 2 copper layers, 84.2 x 107.3 mm, 78 parts, among them J1 Conn_02x25_Counter_Clockwise, SW1 1U, SW10 1U, SW11 1U, SW12 1U, SW13 1U, SW14 1U, SW15 1U, SW16 2U, SW17 2U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

Commit message: revA production ready
Connections:
- net Net-(J1-Pad33) renamed /COL8
- net Net-(J1-Pad35) renamed /COL10
- net Net-(J1-Pad36) renamed /COL11
- net Net-(J1-Pad37) renamed /COL12
- net Net-(J1-Pad38) renamed /COL13
- net Net-(J1-Pad39) renamed /COL14
- net Net-(J1-Pad40) renamed /COL15
- J1 pad 34: /LED_DAT1 -> /COL9
- J1 pad 41: Net-(J1-Pad41) -> /LED_DAT1
Routing:
- net /LED_DAT1: track 126.9 -> 124.0 mm
Other:
- board text added: "JLCJLCJLC"
- board text added: "Licensed under CERN-OHL-P v2"
- board text removed: "Licensed under CERN-OHL-W v2"
